File: SX1276_SCH_Roy/SX1276.kicad_sch (KiCad schematic)
At the start: 23 parts, among them J1 Conn_Coaxial, U1 SX1276, U2 PE4259, Y1 32MHz

Commit message: Rename stuff for Main Chip
Connections:
- net RESET: no longer MCU_Header1.7 (Pin_7)
- net +3V3 renamed +3.3V
- net DI00 renamed SX1276_DI00_N
- net MISO renamed SX1276_MISO_N
- net MOSI renamed SX1276_MOSI_N
- net NSS renamed SX1276_NSS_N
- net SCK renamed SX1276_SCK_N
- new net SX1276_RESET_N: MCU_Header1.7 (Pin_7)
