File: Batteri lader real/batteri lader pcb.kicad_sch (KiCad schematic)
At the start: 10 parts, among them U1 BQ24074RGT

Commit message: AHHHHHHH
Parts:
- added C3: 10uF, symbol Device:C_Small
- C1: value 1μF -> 1uF
- C2: value 4.7μF -> 4.7uF
- R1, R2, R3: value 10kΩ -> 10k
- R4: value 1.13kΩ -> 1.13k
- R5: value 1.18kΩ -> 1.18k
Connections:
- net GND: now also C3.1
- net battery +: now also C3.2
Changed lines of the file:
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@@
 	(paper "A4")
+	(junction
+		(at 138.43 107.95)
+		(diameter 0)
+		(color 0 0 0 0)
+	)
 	(junction
 		(at 176.53 82.55)
@@
 	)
 	(junction
+		(at 182.88 90.17)
+		(diameter 0)
+		(color 0 0 0 0)
+	)
+	(junction
 		(at 154.94 82.55)
 		(diameter 0)
@@
 	(wire
 		(pts
+			(xy 182.88 90.17) (xy 193.04 90.17)
+		)
+		(stroke
+			(width 0)
+			(type default)
+		)
+	)
+	(wire
+		(pts
+			(xy 142.24 114.3) (xy 142.24 115.57)
+		)
+		(stroke
+			(width 0)
+			(type default)
+		)
+	)
+	(wire
+		(pts
 			(xy 161.29 99.06) (xy 161.29 100.33)
 		)
@@
 	(wire
 		(pts
+			(xy 142.24 107.95) (xy 138.43 107.95)
+		)
+		(stroke
+			(width 0)
+			(type default)
+		)
+	)
+	(wire
+		(pts
 			(xy 160.02 95.25) (xy 163.83 95.25)
 		)
@@
 	(wire
 		(pts
+			(xy 182.88 115.57) (xy 142.24 115.57)
+		)
+		(stroke
+			(width 0)
+			(type default)
+		)
+	)
+	(wire
+		(pts
 			(xy 151.13 102.87) (xy 152.4 102.87)
 		)
@@
 	(wire
 		(pts
+			(xy 142.24 107.95) (xy 142.24 109.22)
+		)
+		(stroke
+			(width 0)
+			(type default)
+		)
+	)
+	(wire
+		(pts
 			(xy 138.43 69.85) (xy 138.43 77.47)
 		)
@@
 	(wire
 		(pts
-			(xy 151.13 90.17) (xy 168.91 90.17)
+			(xy 151.13 90.17) (xy 182.88 90.17)
+		)
+		(stroke
+			(width 0)
+			(type default)
+		)
+	)
+	(wire
+		(pts
+			(xy 182.88 90.17) (xy 182.88 115.57)
 		)
 		(stroke
@@
 	)
 	(label "(can replace LED with GPIO mcu)"
-		(at 148.59 111.76 0)
+		(at 151.13 110.49 0)
 		(effects
 			(font
@@
 		)
 	)
+	(label "4.35V_to_10.5V"
+		(at 137.16 121.92 0)
+		(effects
+			(font
+				(size 0.75 0.75)
+			)
+			(justify left bottom)
+		)
+	)
+	(label "4.35V_to_10.5V"
+		(at 142.24 66.04 0)
+		(effects
+			(font
+				(size 0.75 0.75)
+			)
+			(justify left bottom)
+		)
+	)
 	(label "battery +"
-		(at 160.02 90.17 0)
+		(at 184.15 90.17 0)
 		(effects
 			(font
@@
 			)
 			(justify left bottom)
+		)
+	)
+	(symbol
+		(lib_id "Device:C_Small")
+		(at 142.24 111.76 0)
+		(unit 1)
+		(body_style 1)
+		(exclude_from_sim no)
+		(in_bom yes)
+		(on_board yes)
+		(in_pos_files yes)
+		(dnp no)
+		(fields_autoplaced yes)
+		(property "Reference" "C3"
+			(at 144.78 110.4962 0)
+			(show_name no)
+			(do_not_autoplace no)
+			(effects
+				(font
+					(size 1.27 1.27)
+				)
+				(justify left)
+			)
+		)
+		(property "Value" "10uF"
+			(at 144.78 113.0362 0)
+			(show_name no)
+			(do_not_autoplace no)
+			(effects
+				(font
+					(size 1.27 1.27)
+				)
+				(justify left)
+			)
+		)
+		(property "Footprint" ""
+			(at 142.24 111.76 0)
+			(hide yes)
+			(show_name no)
+			(do_not_autoplace no)
+			(effects
+				(font
+					(size 1.27 1.27)
+				)
+			)
+		)
+		(property "Datasheet" ""
+			(at 142.24 111.76 0)
+			(hide yes)
+			(show_name no)
+			(do_not_autoplace no)
+			(effects
+				(font
+					(size 1.27 1.27)
+				)
+			)
+		)
+		(property "Description" "Unpolarized capacitor, small symbol"
+			(at 142.24 111.76 0)
+			(hide yes)
+			(show_name no)
+			(do_not_autoplace no)
+			(effects
+				(font
+					(size 1.27 1.27)
+				)
+			)
+		)
+		(pin "2"
+		)
+		(pin "1"
+		)
+		(instances
+			(project "batteri lader pcb"
+				(path "/f0f8d5a6-dff9-4180-8a23-3182a588a69e"
+					(reference "C3")
+					(unit 1)
+				)
+			)
 		)
 	)
@@
 			)
 		)
-		(property "Value" "10kΩ"
+		(property "Value" "10k"
 			(at 159.258 93.218 90)
 			(show_name no)
@@
 			)
 		)
-		(property "Value" "1.13kΩ"
+		(property "Value" "1.13k"
 			(at 123.698 105.156 90)
 			(show_name no)
@@
 			)
 		)
-		(property "Value" "1.18kΩ"
+		(property "Value" "1.18k"
 			(at 122.682 98.044 90)
 			(show_name no)
@@
 			)
 		)
-		(property "Value" "4.7μF"
+		(property "Value" "4.7uF"
 			(at 157.48 86.3662 0)
 			(show_name no)
@@
 			)
 		)
-		(property "Value" "10kΩ"
-			(at 158.496 105.41 90)
+		(property "Value" "10k"
+			(at 158.75 105.156 90)
 			(show_name no)
 			(do_not_autoplace no)
@@
 		(dnp no)
 		(property "Reference" "U1"
-			(at 140.97 74.168 0)
+			(at 140.208 79.248 0)
 			(show_name no)
 			(do_not_autoplace no)
@@
 		)
 		(property "Value" "BQ24074RGT"
-			(at 140.208 77.47 0)
+			(at 133.096 86.106 0)
 			(show_name no)
 			(do_not_autoplace no)
@@
 			)
 		)
-		(property "Value" "1μF"
+		(property "Value" "1uF"
 			(at 137.16 113.0362 0)
 			(show_name no)
@@
 			)
 		)
-		(property "Value" "10kΩ"
+		(property "Value" "10k"
 			(at 159.258 98.298 90)
 			(show_name no)

Commit message: fiksa og triksa lit
Other:
- note added: "I_CHARGE = 890 / R_ISET"
Changed lines of the file:
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@@
 	(generator_version "10.0")
 	(paper "A4")
+	(text "I_CHARGE = 890 / R_ISET"
+		(exclude_from_sim no)
+		(at 120.142 106.68 0)
+		(effects
+			(font
+				(size 0.5 0.5)
+			)
+		)
+	)
 	(junction
 		(at 138.43 107.95)
@@
 		(property "Reference" "U1"
 			(at 140.208 79.248 0)
-			(show_name no)
-			(do_not_autoplace no)
+			(hide yes)
+			(show_name no)
+			(do_not_autoplace no)
