File: GPS pcb real/gps pcb/gps pcb.kicad_pcb (KiCad board)
At the start: 2 copper layers, 2 parts, among them U1 MIA-M10Q

Commit message: gps
Parts:
- moved U1 98.1 mm to (149.5, 100.5)
- moved D1 86.3 mm to (153.9, 109.0)
Changed lines of the file:
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@@
 	(footprint "Diode_THT:D_DO-35_SOD27_P7.62mm_Horizontal"
 		(layer "F.Cu")
-		(at 234.075 140.775)
+		(at 153.88 109)
 		(descr "Diode, DO-35_SOD27 series, Axial, Horizontal, pin pitch=7.62mm, length*diameter=4*2mm^2, http://www.diodes.com/_files/packages/DO-35.pdf")
 		(tags "Diode DO-35_SOD27 series Axial Horizontal pin pitch 7.62mm  length 4mm diameter 2mm")
@@
 	(footprint "Package_LGA:ublox_LGA-53_4.5x4.5mm_Layout9x9_P0.5mm"
 		(layer "F.Cu")
-		(at 236.275 146.325)
+		(at 149.5 100.5)
 		(descr "ublox MIA SoC Module, 4.5x4.5mm, 53 Ball, 9x9 Layout, 0.5mm Pitch, https://content.u-blox.com/sites/default/files/documents/MIA-M10Q_IntegrationManual_UBX-21028173.pdf#page=82")
 		(tags "LGA 53 0.5 ublox_MIA-M-LGA53")
