File: GPS pcb real/gps pcb/gps pcb.kicad_sch (KiCad schematic)
At the start: 7 parts, among them U1 MIA-M10Q

Commit message: fiksa filsystemer (ish)
Parts:
- renumbered BT1 to GPS_BT1
Connections:
- net GPS RESET renamed GPS_RESET_N
- net GPS TIMEPULSE renamed GPS_TIMEPULSE_N
- net GPS WAKE renamed GPS_WAKE_N
- net MCU RX renamed MCU_RX_N
- net MCU TX renamed MCU_TX_N
Changed lines of the file:
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@@
 	(wire
 		(pts
-			(xy 114.3 101.6) (xy 132.08 101.6)
+			(xy 110.49 101.6) (xy 132.08 101.6)
+		)
+		(stroke
+			(width 0)
+			(type default)
+		)
+	)
+	(wire
+		(pts
+			(xy 114.3 83.82) (xy 132.08 83.82)
 		)
 		(stroke
@@
 	(wire
 		(pts
-			(xy 142.24 55.88) (xy 114.3 55.88)
+			(xy 142.24 55.88) (xy 110.49 55.88)
 		)
 		(stroke
@@
 	(wire
 		(pts
-			(xy 116.84 83.82) (xy 132.08 83.82)
+			(xy 110.49 55.88) (xy 110.49 101.6)
 		)
 		(stroke
@@
 	(wire
 		(pts
-			(xy 114.3 55.88) (xy 114.3 101.6)
-		)
-		(stroke
-			(width 0)
-			(type default)
-		)
-	)
-	(wire
-		(pts
 			(xy 116.84 81.28) (xy 132.08 81.28)
 		)
@@
 		)
 	)
-	(label "MCU RX"
+	(label "MCU_RX_N"
 		(at 116.84 73.66 0)
 		(effects
@@
 		)
 	)
-	(label "MCU TX"
+	(label "MCU_TX_N"
 		(at 116.84 76.2 0)
 		(effects
@@
 		)
 	)
-	(label "GPS WAKE"
+	(label "GPS_WAKE_N"
 		(at 116.84 81.28 0)
 		(effects
@@
 		)
 	)
-	(label "GPS TIMEPULSE"
-		(at 116.84 83.82 0)
+	(label "GPS_TIMEPULSE_N"
+		(at 114.3 83.82 0)
 		(effects
 			(font
@@
 		)
 	)
-	(label "GPS RESET"
+	(label "GPS_RESET_N"
 		(at 116.84 96.52 0)
 		(effects
@@
 		(dnp no)
 		(fields_autoplaced yes)
-		(property "Reference" "BT1"
+		(property "Reference" "GPS_BT1"
 			(at 157.48 26.6699 90)
 			(show_name no)
@@
 			(project "gps pcb"
 				(path "/8ebbdced-8093-4286-89ad-c0afecb178dd"
-					(reference "BT1")
+					(reference "GPS_BT1")
 					(unit 1)
 				)

Commit message: AHHHHHHH
Parts:
- added J1: Conn_Coaxial, symbol Connector:Conn_Coaxial
- C2: value 10µF -> 10uF
Connections:
- net GND: now also J1.2 (Ext)
- net at U1.B9 (RF_IN): now also J1.1 (In)
Changed lines of the file:
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@@
+	(wire
+		(pts
+			(xy 162.56 68.58) (xy 173.99 68.58)
+		)
+		(stroke
+			(width 0)
+			(type default)
+		)
+	)
 	(wire
 		(pts
@@
 		)
 		(property "Value" "MIA-M10Q"
-			(at 150.114 115.57 0)
+			(at 150.368 115.57 0)
 			(show_name no)
 			(do_not_autoplace no)
@@
 	)
 	(symbol
+		(lib_id "power:GND")
+		(at 179.07 73.66 0)
+		(unit 1)
+		(body_style 1)
+		(exclude_from_sim no)
+		(in_bom yes)
+		(on_board yes)
+		(in_pos_files yes)
+		(dnp no)
+		(fields_autoplaced yes)
+		(property "Reference" "#PWR04"
+			(at 179.07 80.01 0)
+			(hide yes)
+			(show_name no)
+			(do_not_autoplace no)
+			(effects
+				(font
+					(size 1.27 1.27)
+				)
+			)
+		)
+		(property "Value" "GND"
+			(at 179.07 78.74 0)
+			(show_name no)
+			(do_not_autoplace no)
+			(effects
+				(font
+					(size 1.27 1.27)
+				)
+			)
+		)
+		(property "Footprint" ""
+			(at 179.07 73.66 0)
+			(hide yes)
+			(show_name no)
+			(do_not_autoplace no)
+			(effects
+				(font
+					(size 1.27 1.27)
+				)
+			)
+		)
+		(property "Datasheet" ""
+			(at 179.07 73.66 0)
+			(hide yes)
+			(show_name no)
+			(do_not_autoplace no)
+			(effects
+				(font
+					(size 1.27 1.27)
+				)
+			)
+		)
+		(property "Description" "Power symbol creates a global label with name \"GND\" , ground"
+			(at 179.07 73.66 0)
+			(hide yes)
+			(show_name no)
+			(do_not_autoplace no)
+			(effects
+				(font
+					(size 1.27 1.27)
+				)
+			)
+		)
+		(pin "1"
+		)
+		(instances
+			(project "gps pcb"
+				(path "/8ebbdced-8093-4286-89ad-c0afecb178dd"
+					(reference "#PWR04")
+					(unit 1)
+				)
+			)
+		)
+	)
+	(symbol
 		(lib_id "Connector_Generic:Conn_01x02")
 		(at 152.4 27.94 90)
@@
 			)
 		)
-		(property "Value" "10µF"
+		(property "Value" "10uF"
 			(at 146.812 50.292 0)
 			(show_name no)
@@
 					(unit 1)
 				)
+			)
+		)
+	)
+	(symbol
+		(lib_id "Connector:Conn_Coaxial")
+		(at 179.07 68.58 0)
+		(unit 1)
+		(body_style 1)
+		(exclude_from_sim no)
+		(in_bom yes)
+		(on_board yes)
+		(in_pos_files yes)
+		(dnp no)
+		(fields_autoplaced yes)
+		(property "Reference" "J1"
+			(at 182.88 67.6031 0)
+			(show_name no)
+			(do_not_autoplace no)
+			(effects
+				(font
+					(size 1.27 1.27)
+				)
+				(justify left)
+			)
+		)
+		(property "Value" "Conn_Coaxial"
+			(at 182.88 70.1431 0)
+			(show_name no)
+			(do_not_autoplace no)
+			(effects
+				(font
+					(size 1.27 1.27)
+				)
+				(justify left)
+			)
+		)
+		(property "Footprint" ""
+			(at 179.07 68.58 0)
+			(hide yes)
+			(show_name no)
+			(do_not_autoplace no)
+			(effects
+				(font
+					(size 1.27 1.27)
+				)
+			)
+		)
+		(property "Datasheet" ""
+			(at 179.07 68.58 0)
+			(hide yes)
+			(show_name no)
+			(do_not_autoplace no)
+			(effects
+				(font
+					(size 1.27 1.27)
+				)
+			)
+		)
+		(property "Description" "coaxial connector (BNC, SMA, SMB, SMC, Cinch/RCA, LEMO, ...)"
+			(at 179.07 68.58 0)
+			(hide yes)
+			(show_name no)
+			(do_not_autoplace no)
+			(effects
+				(font
+					(size 1.27 1.27)
+				)
+			)
+		)
+		(pin "2"
+		)
+		(pin "1"
+		)
+		(instances
+			(project "gps pcb"
+				(path "/8ebbdced-8093-4286-89ad-c0afecb178dd"
+					(reference "J1")
+					(unit 1)
+				)

Commit message: fiksa og triksa lit
Parts:
- removed C1: 100nF, symbol Device:C
- removed C2: 10uF, symbol Device:C
Connections:
- net +3.3VADC: now also U1.B1 (VCC), U1.J4 (V_IO)
- now unconnected: U1.J6 (VIO_SEL)
- no-connect marks 12 -> 13
Changed lines of the file:
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@@
-	)
-	(junction
-		(at 142.24 55.88)
-		(diameter 0)
-		(color 0 0 0 0)
 	)
 	(junction
@@
 	)
 	(junction
-		(at 143.51 44.45)
-		(diameter 0)
-		(color 0 0 0 0)
-	)
-	(junction
 		(at 143.51 55.88)
 		(diameter 0)
@@
 	)
 	(no_connect
+		(at 132.08 101.6)
+	)
+	(no_connect
 		(at 162.56 109.22)
 	)
@@
 	(wire
 		(pts
-			(xy 110.49 101.6) (xy 132.08 101.6)
+			(xy 143.51 55.88) (xy 144.78 55.88)
+		)
+		(stroke
+			(width 0)
+			(type default)
+		)
+	)
+	(wire
+		(pts
+			(xy 143.51 44.45) (xy 143.51 55.88)
 		)
 		(stroke
@@
 	(wire
 		(pts
-			(xy 140.97 44.45) (xy 143.51 44.45)
-		)
-		(stroke
-			(width 0)
-			(type default)
-		)
-	)
-	(wire
-		(pts
 			(xy 116.84 76.2) (xy 132.08 76.2)
 		)
@@
 	(wire
 		(pts
-			(xy 142.24 55.88) (xy 110.49 55.88)
-		)
-		(stroke
-			(width 0)
-			(type default)
-		)
-	)
-	(wire
-		(pts
 			(xy 144.78 55.88) (xy 144.78 58.42)
 		)
@@
 	(wire
 		(pts
-			(xy 143.51 55.88) (xy 144.78 55.88)
-		)
-		(stroke
-			(width 0)
-			(type default)
-		)
-	)
-	(wire
-		(pts
 			(xy 116.84 96.52) (xy 132.08 96.52)
 		)
@@
 	(wire
 		(pts
-			(xy 143.51 49.53) (xy 143.51 55.88)
-		)
-		(stroke
-			(width 0)
-			(type default)
-		)
-	)
-	(wire
-		(pts
 			(xy 116.84 73.66) (xy 132.08 73.66)
 		)
@@
 	(wire
 		(pts
-			(xy 110.49 55.88) (xy 110.49 101.6)
-		)
-		(stroke
-			(width 0)
-			(type default)
-		)
-	)
-	(wire
-		(pts
 			(xy 152.4 55.88) (xy 152.4 48.26)
 		)
@@
 		(pts
 			(xy 116.84 81.28) (xy 132.08 81.28)
-		)
-		(stroke
-			(width 0)
-			(type default)
-		)
-	)
-	(wire
-		(pts
-			(xy 143.51 44.45) (xy 146.05 44.45)
-		)
-		(stroke
-			(width 0)
-			(type default)
-		)
-	)
-	(wire
-		(pts
-			(xy 140.97 52.07) (xy 146.05 52.07)
 		)
 		(stroke
@@
 	)
 	(symbol
-		(lib_id "Device:C")
-		(at 140.97 48.26 0)
-		(unit 1)
-		(body_style 1)
-		(exclude_from_sim no)
-		(in_bom yes)
-		(on_board yes)
-		(in_pos_files yes)
-		(dnp no)
-		(property "Reference" "C1"
-			(at 137.414 45.974 0)
-			(show_name no)
-			(do_not_autoplace no)
-			(effects
-				(font
-					(size 1.27 1.27)
-				)
-				(justify left)
-			)
-		)
-		(property "Value" "100nF"
-			(at 134.62 50.038 0)
-			(show_name no)
-			(do_not_autoplace no)
-			(effects
-				(font
-					(size 1.27 1.27)
-				)
-				(justify left)
-			)
-		)
-		(property "Footprint" ""
-			(at 141.9352 52.07 0)
-			(hide yes)
-			(show_name no)
-			(do_not_autoplace no)
-			(effects
-				(font
-					(size 1.27 1.27)
-				)
-			)
-		)
-		(property "Datasheet" ""
-			(at 140.97 48.26 0)
-			(hide yes)
-			(show_name no)
-			(do_not_autoplace no)
-			(effects
-				(font
-					(size 1.27 1.27)
-				)
-			)
-		)
-		(property "Description" "Unpolarized capacitor"
-			(at 140.97 48.26 0)
-			(hide yes)
-			(show_name no)
-			(do_not_autoplace no)
-			(effects
-				(font
-					(size 1.27 1.27)
-				)
-			)
-		)
-		(pin "1"
-		)
-		(pin "2"
-		)
-		(instances
-			(project "gps pcb"
-				(path "/8ebbdced-8093-4286-89ad-c0afecb178dd"
-					(reference "C1")
-					(unit 1)
-				)
-			)
-		)
-	)
-	(symbol
 		(lib_id "power:GND")
 		(at 147.32 119.38 0)
@@
 					(unit 1)
 				)
-			)
-		)
-	)
-	(symbol
-		(lib_id "Device:C")
-		(at 146.05 48.26 0)
-		(unit 1)
-		(body_style 1)
-		(exclude_from_sim no)
-		(in_bom yes)
-		(on_board yes)
-		(in_pos_files yes)
-		(dnp no)
-		(property "Reference" "C2"
-			(at 147.32 46.228 0)
-			(show_name no)
-			(do_not_autoplace no)
-			(effects
-				(font
-					(size 1.27 1.27)
-				)
-				(justify left)
-			)
-		)
-		(property "Value" "10uF"
-			(at 146.812 50.292 0)
-			(show_name no)
-			(do_not_autoplace no)
-			(effects
-				(font
-					(size 1.27 1.27)
-				)
-				(justify left)
-			)
-		)
-		(property "Footprint" ""
-			(at 147.0152 52.07 0)
-			(hide yes)
-			(show_name no)
-			(do_not_autoplace no)
-			(effects
-				(font
-					(size 1.27 1.27)
-				)
-			)
-		)
-		(property "Datasheet" ""
-			(at 146.05 48.26 0)
-			(hide yes)
-			(show_name no)
-			(do_not_autoplace no)
-			(effects
-				(font
-					(size 1.27 1.27)
-				)
-			)
-		)
-		(property "Description" "Unpolarized capacitor"
-			(at 146.05 48.26 0)
-			(hide yes)
-			(show_name no)
-			(do_not_autoplace no)
-			(effects
-				(font
-					(size 1.27 1.27)
-				)
-			)
-		)
-		(pin "1"
-		)
-		(pin "2"
-		)
-		(instances
-			(project "gps pcb"
-				(path "/8ebbdced-8093-4286-89ad-c0afecb178dd"
-					(reference "C2")
-					(unit 1)
-				)

Commit message: gps
Connections:
- net at D1.1 (K), U1.J5 (V_BCKP): no longer C3.1, D1.2 (A)
- new net: C3.1, D1.2 (A)
Changed lines of the file:
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@@
 	(paper "A4")
-	(junction
-		(at 152.4 55.88)
-		(diameter 0)
-		(color 0 0 0 0)
-	)
-	(junction
-		(at 152.4 48.26)
-		(diameter 0)
-		(color 0 0 0 0)
-	)
 	(junction
 		(at 143.51 55.88)
@@
 		)
 		(stroke
-			(width 0)
-			(type default)
-		)
-	)
-	(wire
-		(pts
-			(xy 152.4 55.88) (xy 152.4 48.26)
-		)
-		(stroke
