File: MCU/MCU_basics/bigBoi/radio.kicad_sch (KiCad schematic)
At the start: 22 parts, among them J1 Conn_Coaxial, U3 SX1276, U4 PE4259, Y2 32MHz

Commit message: footprints assigned
Parts:
- removed Y2: 32MHz, symbol Device:Crystal
- added Y2: 32MHz, Crystal:Crystal_SMD_3225-4Pin_3.2x2.5mm, symbol Device:Crystal_GND24
- U3: footprint Package_DFN_QFN:QFN-28-1EP_6x6mm_P0.65mm_EP4.8x4.8mm -> Nebula-footprints:QFN65P600X600X100-29N
- U4: footprint PE4259:SOT65P215X110-6N -> Nebula-footprints:SOT65P215X110-6N
Connections:
- net GND: now also Y2.2 (G), Y2.4 (G)
- net at C47.1, U3.6 (XTB): now also Y2.3
- net at C28.1, U3.5 (XTA): now also Y2.1
Changed lines of the file:
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@@
 	(wire
 		(pts
+			(xy 116.84 78.74) (xy 124.46 78.74)
+		)
+		(stroke
+			(width 0)
+			(type default)
+		)
+	)
+	(wire
+		(pts
 			(xy 173.99 101.6) (xy 171.45 101.6)
 		)
@@
 	(wire
 		(pts
-			(xy 120.65 86.36) (xy 121.92 86.36)
-		)
-		(stroke
-			(width 0)
-			(type default)
-		)
-	)
-	(wire
-		(pts
 			(xy 125.73 59.69) (xy 125.73 63.5)
 		)
@@
 	(wire
 		(pts
-			(xy 227.33 83.82) (xy 224.79 83.82)
+			(xy 116.84 86.36) (xy 121.92 86.36)
 		)
 		(stroke
@@
 	(wire
 		(pts
-			(xy 124.46 85.09) (xy 121.92 85.09)
+			(xy 227.33 83.82) (xy 224.79 83.82)
 		)
 		(stroke
@@
 	(wire
 		(pts
-			(xy 209.55 109.22) (xy 218.44 109.22)
+			(xy 124.46 85.09) (xy 121.92 85.09)
 		)
 		(stroke
@@
 	(wire
 		(pts
-			(xy 168.91 104.14) (xy 207.01 104.14)
+			(xy 209.55 109.22) (xy 218.44 109.22)
 		)
 		(stroke
@@
 	(wire
 		(pts
-			(xy 163.83 59.69) (xy 163.83 62.23)
+			(xy 168.91 104.14) (xy 207.01 104.14)
 		)
 		(stroke
@@
 	(wire
 		(pts
-			(xy 111.76 90.17) (xy 111.76 96.52)
+			(xy 163.83 59.69) (xy 163.83 62.23)
 		)
 		(stroke
@@
 	(wire
 		(pts
-			(xy 217.17 92.71) (xy 218.44 92.71)
+			(xy 111.76 90.17) (xy 111.76 96.52)
 		)
 		(stroke
@@
 	(wire
 		(pts
-			(xy 120.65 78.74) (xy 124.46 78.74)
+			(xy 217.17 92.71) (xy 218.44 92.71)
 		)
 		(stroke
@@
 			)
 		)
-		(property "Footprint" "Package_DFN_QFN:QFN-28-1EP_6x6mm_P0.65mm_EP4.8x4.8mm"
+		(property "Footprint" "Nebula-footprints:QFN65P600X600X100-29N"
 			(at 139.7 104.14 0)
 			(hide yes)
@@
 	)
 	(symbol
-		(lib_id "Device:Crystal")
-		(at 120.65 82.55 90)
-		(unit 1)
-		(body_style 1)
-		(exclude_from_sim no)
-		(in_bom yes)
-		(on_board yes)
-		(in_pos_files yes)
-		(dnp no)
-		(property "Reference" "Y2"
-			(at 115.062 81.28 90)
-			(show_name no)
-			(do_not_autoplace no)
-			(effects
-				(font
-					(size 1.27 1.27)
-				)
-				(justify right)
-			)
-		)
-		(property "Value" "32MHz"
-			(at 111.252 83.82 90)
-			(show_name no)
-			(do_not_autoplace no)
-			(effects
-				(font
-					(size 1.27 1.27)
-				)
-				(justify right)
-			)
-		)
-		(property "Footprint" ""
-			(at 120.65 82.55 0)
-			(hide yes)
-			(show_name no)
-			(do_not_autoplace no)
-			(effects
-				(font
-					(size 1.27 1.27)
-				)
-			)
-		)
-		(property "Datasheet" ""
-			(at 120.65 82.55 0)
-			(hide yes)
-			(show_name no)
-			(do_not_autoplace no)
-			(effects
-				(font
-					(size 1.27 1.27)
-				)
-			)
-		)
-		(property "Description" "Two pin crystal"
-			(at 120.65 82.55 0)
-			(hide yes)
-			(show_name no)
-			(do_not_autoplace no)
-			(effects
-				(font
-					(size 1.27 1.27)
-				)
-			)
-		)
-		(pin "2"
-		)
-		(pin "1"
-		)
-		(instances
-			(project "bigBoi"
-				(path "/0a118c22-2522-42a6-b7a6-70c79326ece4/f88a4f50-bdfc-44db-bd06-a2b26240335b"
-					(reference "Y2")
-					(unit 1)
-				)
-			)
-		)
-	)
-	(symbol
 		(lib_id "power:GND")
 		(at 104.14 77.47 270)
@@
 	(symbol
 		(lib_id "power:GND")
+		(at 111.76 82.55 270)
+		(unit 1)
+		(body_style 1)
+		(exclude_from_sim no)
+		(in_bom yes)
+		(on_board yes)
+		(in_pos_files yes)
+		(dnp no)
+		(property "Reference" "#PWR078"
+			(at 105.41 82.55 0)
+			(hide yes)
+			(show_name no)
+			(do_not_autoplace no)
+			(effects
+				(font
+					(size 1.27 1.27)
+				)
+			)
+		)
+		(property "Value" "GND"
+			(at 111.76 84.836 90)
+			(hide yes)
+			(show_name no)
+			(do_not_autoplace no)
+			(effects
+				(font
+					(size 1.27 1.27)
+				)
+				(justify right)
+			)
+		)
+		(property "Footprint" ""
+			(at 111.76 82.55 0)
+			(hide yes)
+			(show_name no)
+			(do_not_autoplace no)
+			(effects
+				(font
+					(size 1.27 1.27)
+				)
+			)
+		)
+		(property "Datasheet" ""
+			(at 111.76 82.55 0)
+			(hide yes)
+			(show_name no)
+			(do_not_autoplace no)
+			(effects
+				(font
+					(size 1.27 1.27)
+				)
+			)
+		)
+		(property "Description" "Power symbol creates a global label with name \"GND\" , ground"
+			(at 111.76 82.55 0)
+			(hide yes)
+			(show_name no)
+			(do_not_autoplace no)
+			(effects
+				(font
+					(size 1.27 1.27)
+				)
+			)
+		)
+		(pin "1"
+		)
+		(instances
+			(project "bigBoi"
+				(path "/0a118c22-2522-42a6-b7a6-70c79326ece4/f88a4f50-bdfc-44db-bd06-a2b26240335b"
+					(reference "#PWR078")
+					(unit 1)
+				)
+			)
+		)
+	)
+	(symbol
+		(lib_id "power:GND")
 		(at 135.89 127 0)
 		(unit 1)
@@
 	)
 	(symbol
+		(lib_id "Device:Crystal_GND24")
+		(at 116.84 82.55 270)
+		(unit 1)
+		(body_style 1)
+		(exclude_from_sim no)
+		(in_bom yes)
+		(on_board yes)
+		(in_pos_files yes)
+		(dnp no)
+		(property "Reference" "Y2"
+			(at 115.316 73.152 90)
+			(show_name no)
+			(do_not_autoplace no)
+			(effects
+				(font
+					(size 1.27 1.27)
+				)
+				(justify left)
+			)
+		)
+		(property "Value" "32MHz"
+			(at 113.03 75.184 90)
+			(show_name no)
+			(do_not_autoplace no)
+			(effects
+				(font
+					(size 1.27 1.27)
+				)
+				(justify left)
+			)
+		)
+		(property "Footprint" "Crystal:Crystal_SMD_3225-4Pin_3.2x2.5mm"
+			(at 116.84 82.55 0)
+			(hide yes)
+			(show_name no)
+			(do_not_autoplace no)
+			(effects
+				(font
+					(size 1.27 1.27)
+				)
+			)
+		)
+		(property "Datasheet" ""
+			(at 116.84 82.55 0)
+			(hide yes)
+			(show_name no)
+			(do_not_autoplace no)
+			(effects
+				(font
+					(size 1.27 1.27)
+				)
+			)
+		)
+		(property "Description" "Four pin crystal, GND on pins 2 and 4"
+			(at 116.84 82.55 0)
+			(hide yes)
+			(show_name no)
+			(do_not_autoplace no)
+			(effects
+				(font
+					(size 1.27 1.27)
+				)
+			)
+		)
+		(property private "KLC_S3.3" "The rectangle is not a symbol body but a graphical element"
+			(at 104.14 82.55 0)
+			(hide yes)
+			(show_name yes)
+			(do_not_autoplace no)
+			(effects
+				(font
+					(size 1.27 1.27)
+				)
+			)
+		)
+		(property private "KLC_S4.1" "Some pins are on 50mil grid to make the symbol small"
+			(at 101.6 82.55 0)
+			(hide yes)
+			(show_name yes)
+			(do_not_autoplace no)
+			(effects
+				(font
+					(size 1.27 1.27)
+				)
+			)
+		)
+		(pin "3"
+		)
+		(pin "1"
+		)
+		(pin "2"
+		)
+		(pin "4"
+		)
+		(instances
+			(project "bigBoi"
+				(path "/0a118c22-2522-42a6-b7a6-70c79326ece4/f88a4f50-bdfc-44db-bd06-a2b26240335b"
+					(reference "Y2")
+					(unit 1)
+				)
+			)
+		)
+	)
+	(symbol
 		(lib_id "Device:C_Small")
 		(at 173.99 91.44 180)
@@
 			)
 		)
-		(property "Footprint" "PE4259:SOT65P215X110-6N"
+		(property "Footprint" "Nebula-footprints:SOT65P215X110-6N"
 			(at 231.14 106.68 0)
 			(hide yes)
