File: MCU/MCU_basics/bigBoi/presTemp.kicad_sch (KiCad schematic)
At the start: 3 parts, among them IC1 BMP390

Commit message: most footprints assigned
Parts:
- IC1: footprint BMP390:BMP390 -> Nebula-footprints:BMP390
Changed lines of the file:
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@@
 			)
 		)
-		(property "Footprint" "BMP390:BMP390"
+		(property "Footprint" "Nebula-footprints:BMP390"
 			(at 157.48 195.25 0)
 			(hide yes)
