File: MCU/MCU_basics/bigBoi/bigBoi.kicad_pcb (KiCad board)
At the start: 4 copper layers, 70 x 70 mm, 97 parts, among them IC1 BMP390, J1 Conn_Coaxial, J2 Conn_Coaxial, J3 DM3AT-SF-PEJM5_40_, J4 Conn_01x05, J5 Conn_01x04, J6 Conn_01x06, J7 USB_B_Micro, SW1 Boot Switch, U1 STM32F469NIHx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

Commit message: SX1276 layout
Parts:
- C30: moved to B.Cu
- Y1, Y3: footprint Crystal:Crystal_SMD_3225-4Pin_3.2x2.5mm_HandSoldering -> Crystal:Crystal_SMD_3225-4Pin_3.2x2.5mm
- moved C56 22.4 mm to (115.7, 119.4), turned to 90 degrees
- moved C55 20.1 mm to (113.1, 119.9), turned to 90 degrees
- moved C53 11.3 mm to (111.0, 120.3)
- moved C47 9.55 mm to (101.1, 125.9)
- moved C58 7.92 mm to (119.0, 119.2), turned to 90 degrees
- moved C57 7.71 mm to (119.1, 123.8), turned to -90 degrees
- moved Y2 7.51 mm to (98.4, 124.9), turned to 180 degrees
- moved C52 7.17 mm to (107.7, 119.9), turned to -90 degrees
- moved C54 6.47 mm to (103.4, 124.5)
- moved C51 6.43 mm to (103.4, 122.5)
- moved R2 6.24 mm to (103.4, 126.7)
- moved J1 6.21 mm to (115.5, 127.5)
- moved L3 6.02 mm to (115.2, 120.8)
- moved C28 5.85 mm to (101.1, 124.0)
- moved C14 5.48 mm to (97.8, 98.4), turned to 90 degrees
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Routing:
- net GND: track 14.1 -> 24.7 mm
- net VDDA: track 0.00 -> 2.81 mm, vias 0 -> 2
- net Net-(U1-VREF+): track 4.10 -> 3.12 mm, vias 0 -> 1

Commit message: routing complete
Parts:
- removed D1: 1N914, Diode_THT:D_DO-35_SOD27_P7.62mm_Horizontal
- removed GPS_BT1: CR1220, Battery:BatteryHolder_Keystone_500
- added BT2: Battery, Battery:BatteryHolder_LINX_BAT-HLD-012-SMT, B.Cu at (90.4, 121.5)
- added C60: 1uF, Capacitor_SMD:C_0402_1005Metric, F.Cu at (95.7, 68.9)
- added C61: 100nF, Capacitor_SMD:C_0402_1005Metric, B.Cu at (94.6, 114.4)
- added C62: 100nF, Capacitor_SMD:C_0402_1005Metric, B.Cu at (96.6, 114.5)
- added D3: BAT54, Diode_SMD:D_0402_1005Metric, F.Cu at (95.1, 115.4)
- C35, C40, C41, C43, C45, C46: moved to B.Cu
- moved J4 57.5 mm to (124.1, 125.8), turned to 135 degrees
- moved REF** 45.3 mm to (108.0, 132.0), turned to -90 degrees
- moved REF** 45.3 mm to (76.0, 100.0), turned to -90 degrees
- moved REF** 45.3 mm to (140.0, 100.0)
- moved REF** 45.3 mm to (108.0, 68.0), turned to -90 degrees
- moved J5 40.5 mm to (114.7, 67.6), turned to 70 degrees
- moved J2 15.9 mm to (101.4, 114.5)
- moved U2 11.3 mm to (126.0, 100.0), turned to 180 degrees
- moved J6 11.1 mm to (82.3, 93.7)
- moved U5 10.8 mm to (95.6, 111.6)
- moved J7 9.62 mm to (137.0, 91.5)
- moved C44 9.54 mm to (101.7, 74.2), turned to -90 degrees
- moved R5 9.42 mm to (93.9, 75.4), turned to 180 degrees
- moved Y3 9.05 mm to (104.4, 73.3), turned to 180 degrees
- moved C42 8.97 mm to (101.7, 72.4), turned to -90 degrees
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Connections:
- C37 pad 1: Net-(D1-A) -> Net-(D3-A)
- U1 pad C12: unconnected-(U1-PD1-PadC12) -> GND
- U5 pad J5: Net-(D1-A) -> Net-(D3-K)
Routing:
- net GND: track 24.7 -> 161.1 mm, vias 35 -> 121
- net /EXT_CS: track 0.00 -> 70.1 mm, vias 0 -> 6
- net GPS_RX_N: track 0.00 -> 61.3 mm, vias 1 -> 6
- net SX1276_MOSI_N: track 0.00 -> 58.7 mm, vias 0 -> 6
- net GPS_TX_N: track 0.00 -> 53.0 mm, vias 1 -> 4
- net GPS_WAKE_N: track 0.00 -> 49.9 mm, vias 0 -> 4
- net +3.3V: track 16.7 -> 66.1 mm, vias 23 -> 56
- net SX1276_RESET_N: track 0.00 -> 49.0 mm, vias 0 -> 4
- net BMP390_MOSI_N: track 0.00 -> 47.9 mm, vias 1 -> 4
- net /PWM_TIM2CH1_SERVOPARA: track 0.00 -> 46.1 mm, vias 0 -> 5
- net BMP390_MISO_N: track 0.00 -> 42.1 mm, vias 1 -> 7
- net Net-(U1-BOOT0): track 0.00 -> 39.7 mm, vias 1 -> 4
- net /SWCLK: track 0.00 -> 37.9 mm, vias 0 -> 5
- net BNO086_WAKE/PS0_N: track 0.00 -> 37.9 mm, vias 0 -> 2
- net BMP390_SCK_N: track 0.00 -> 37.9 mm, vias 1 -> 3
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Other:
- board text added: "(stop looking at my bottom)"
- board text added: "3.3VI"
- board text added: "3.3Vo"
- board text added: "CS"
- board text added: "DRAGONFLY"
- board text added: "F1"
- board text added: "F2"
- board text added: "F3"
- board text added: "F4"
- board text added: "GND"
- board text added: "HI"
- board text added: "LO"
- board text added: "MISO(4)"
- board text added: "MOSI(4)"
- board text added: "NASA|NEBULA|Elvebakken vgs"
- board text added: "NEBULA"
- board text added: "PARA"
- board text added: "SCLK(4)"
- board text added: "SWCLK"
- board text added: "SWDIO"
